File: Linear_Voltage_Regulator_5V.kicad_pcb (KiCad board)
At the start: 2 copper layers, 145 x 45 mm, 8 parts, among them J1 INPUT 7-35V, J2 OUTPUT 5V, U1 L7805CV

Commit message: Task1: ajout rapport + BOM + nettoyage fichiers temporaires
Parts:
- moved C1 16.6 mm to (98.3, 96.0)
- moved C2 16.6 mm to (115.5, 110.5)
- moved C3 16.6 mm to (151.8, 96.0)
- moved J1 16.6 mm to (84.5, 96.0)
- moved J2 16.6 mm to (178.0, 96.0)
- moved R1 16.6 mm to (152.0, 105.9)
- moved R2 16.6 mm to (175.5, 116.0)
- moved U1 16.6 mm to (117.5, 96.0)
Changed lines of the file:
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@@
 	)
 	(paper "A4")
+	(title_block
+		(title "5 V Linear Voltage Regulator")
+		(date "2026-03-14")
+		(rev "1.0")
+		(company "EUTech engineers")
+		(comment 1 "Regulator: L7805CV")
+		(comment 2 "Designer: Assane DIENG ( Electrical Engineering Apprentice)")
+	)
 	(layers
 		(0 "F.Cu" signal)
@@
 			(outputformat 1)
 			(mirror no)
-			(drillshape 1)
+			(drillshape 0)
 			(scaleselection 1)
-			(outputdirectory "")
+			(outputdirectory "./")
 		)
 	)
@@
 	(footprint "Capacitor_THT:CP_Radial_D5.0mm_P2.50mm"
 		(layer "F.Cu")
-		(at 136.294888 90 -90)
+		(at 151.794888 96 -90)
 		(descr "CP, Radial series, Radial, pin pitch=2.50mm, diameter=5mm, height=7mm, Electrolytic Capacitor")
 		(tags "CP Radial series Radial pin pitch 2.50mm diameter 5mm height 7mm Electrolytic Capacitor")
@@
 	(footprint "Capacitor_THT:CP_Radial_D8.0mm_P3.50mm"
 		(layer "F.Cu")
-		(at 82.847349 90 -90)
+		(at 98.347349 96 -90)
 		(descr "CP, Radial series, Radial, pin pitch=3.50mm, diameter=8mm, height=12mm, Electrolytic Capacitor")
 		(tags "CP Radial series Radial pin pitch 3.50mm diameter 8mm height 12mm Electrolytic Capacitor")
@@
 	(footprint "LED_THT:LED_D3.0mm"
 		(layer "F.Cu")
-		(at 160 110)
+		(at 175.5 116)
 		(descr "LED, diameter 3.0mm, 2 pins, generated by kicad-footprint-generator")
 		(tags "LED")
@@
 	(footprint "Connector_PinHeader_2.54mm:PinHeader_1x02_P2.54mm_Vertical"
 		(layer "F.Cu")
-		(at 162.5 90)
+		(at 178 96)
 		(descr "Through hole straight pin header, 1x02, 2.54mm pitch, single row")
 		(tags "Through hole pin header THT 1x02 2.54mm single row")
@@
 	(footprint "Package_TO_SOT_THT:TO-220-3_Vertical"
 		(layer "F.Cu")
-		(at 101.96 89.95)
+		(at 117.46 95.95)
 		(descr "TO-220-3, Vertical, RM 2.54mm, see https://www.vishay.com/docs/66542/to-220-1.pdf, generated with kicad-footprint-generator TO_SOT_THT_generate.py")
 		(tags "TO-220-3 Vertical RM 2.54mm")
@@
 	(footprint "Connector_PinHeader_2.54mm:PinHeader_1x02_P2.54mm_Vertical"
 		(layer "F.Cu")
-		(at 69 90)
+		(at 84.5 96)
 		(descr "Through hole straight pin header, 1x02, 2.54mm pitch, single row")
 		(tags "Through hole pin header THT 1x02 2.54mm single row")
@@
 	(footprint "Resistor_THT:R_Axial_DIN0207_L6.3mm_D2.5mm_P10.16mm_Horizontal"
 		(layer "F.Cu")
-		(at 136.5 99.92 -90)
+		(at 152 105.92 -90)
 		(descr "Resistor, Axial_DIN0207 series, Axial, Horizontal, pin pitch=10.16mm, 0.25W = 1/4W, length*diameter=6.3*2.5mm^2, http://cdn-reichelt.de/documents/datenblatt/B400/1_4W%23YAG.pdf")
 		(tags "Resistor Axial_DIN0207 series Axial Horizontal pin pitch 10.16mm 0.25W = 1/4W length 6.3mm diameter 2.5mm")
@@
 	(footprint "Capacitor_THT:C_Disc_D5.0mm_W2.5mm_P5.00mm"
 		(layer "F.Cu")
-		(at 100 104.5)
+		(at 115.5 110.5)
 		(descr "C, Disc series, Radial, pin pitch=5.00mm, diameter*width=5*2.5mm^2, Capacitor, http://cdn-reichelt.de/documents/datenblatt/B300/DS_KERKO_TC.pdf")
 		(tags "C Disc series Radial pin pitch 5.00mm diameter 5mm width 2.5mm Capacitor")
@@
 	)
 	(segment
-		(start 83 90)
-		(end 83.05 89.95)
+		(start 98.5 96)
+		(end 98.55 95.95)
 		(width 0.2)
 		(layer "F.Cu")
@@
 	)
 	(segment
-		(start 75 103)
-		(end 75 90)
+		(start 90.5 109)
+		(end 90.5 96)
 		(width 0.5)
 		(layer "F.Cu")
@@
 	)
 	(segment
-		(start 95 90)
-		(end 101.91 90)
+		(start 110.5 96)
+		(end 117.41 96)
 		(width 1.5)
 		(layer "F.Cu")
@@
 	)
 	(segment
-		(start 101.91 90)
-		(end 101.96 89.95)
+		(start 117.41 96)
+		(end 117.46 95.95)
 		(width 1.5)
 		(layer "F.Cu")
@@
 	)
 	(segment
-		(start 69 90)
-		(end 75 90)
+		(start 84.5 96)
+		(end 90.5 96)
 		(width 1.5)
 		(layer "F.Cu")
@@
 	)
 	(segment
-		(start 76.5 104.5)
-		(end 75 103)
+		(start 92 110.5)
+		(end 90.5 109)
 		(width 0.5)
 		(layer "F.Cu")
@@
 	)
 	(segment
-		(start 82.847349 90)
-		(end 83 90)
+		(start 98.347349 96)
+		(end 98.5 96)
 		(width 0.2)
 		(layer "F.Cu")
@@
 	)
 	(segment
-		(start 75 90)
-		(end 95 90)
+		(start 90.5 96)
+		(end 110.5 96)
 		(width 1.5)
 		(layer "F.Cu")
@@
 	)
 	(segment
-		(start 100 104.5)
-		(end 76.5 104.5)
+		(start 115.5 110.5)
+		(end 92 110.5)
 		(width 0.5)
 		(layer "F.Cu")
@@
 	)
 	(segment
-		(start 121 100)
-		(end 120 99)
+		(start 136.5 106)
+		(end 135.5 105)
 		(width 0.5)
 		(layer "F.Cu")
@@
 	)
 	(segment
-		(start 107 90)
-		(end 120 90)
+		(start 122.5 96)
+		(end 135.5 96)
 		(width 1.5)
 		(layer "F.Cu")
@@
 	)
 	(segment
-		(start 107.04 89.95)
-		(end 107.04 89.96)
+		(start 122.54 95.95)
+		(end 122.54 95.96)
 		(width 1.5)
 		(layer "F.Cu")
@@
 	)
 	(segment
-		(start 107.04 89.96)
-		(end 107 90)
+		(start 122.54 95.96)
+		(end 122.5 96)
 		(width 1.5)
 		(layer "F.Cu")
@@
 	)
 	(segment
-		(start 136.5 99.92)
-		(end 136.08 99.92)
+		(start 152 105.92)
+		(end 151.58 105.92)
 		(width 0.5)
 		(layer "F.Cu")
@@
 	)
 	(segment
-		(start 136 100)
-		(end 121 100)
+		(start 151.5 106)
+		(end 136.5 106)
 		(width 0.5)
 		(layer "F.Cu")
@@
 	)
 	(segment
-		(start 162.5 90)
-		(end 136.294888 90)
+		(start 178 96)
+		(end 151.794888 96)
 		(width 1.5)
 		(layer "F.Cu")
@@
 	)
 	(segment
-		(start 120 99)
-		(end 120 90)
+		(start 135.5 105)
+		(end 135.5 96)
 		(width 0.5)
 		(layer "F.Cu")
@@
 	)
 	(segment
-		(start 136.08 99.92)
-		(end 136 100)
+		(start 151.58 105.92)
+		(end 151.5 106)
 		(width 0.5)
 		(layer "F.Cu")
@@
 	)
 	(segment
-		(start 136.294888 90)
-		(end 120 90)
+		(start 151.794888 96)
+		(end 135.5 96)
 		(width 1.5)
 		(layer "F.Cu")
@@
 	)
 	(segment
-		(start 107.09 90)
-		(end 107.04 89.95)
+		(start 122.59 96)
+		(end 122.54 95.95)
 		(width 1.5)
 		(layer "B.Cu")
@@
 	)
 	(segment
-		(start 107 89.99)
-		(end 107.04 89.95)
+		(start 122.5 95.99)
+		(end 122.54 95.95)
 		(width 1.5)
 		(layer "B.Cu")
@@
 	)
 	(segment
-		(start 136.244888 89.95)
-		(end 136.294888 90)
+		(start 151.744888 95.95)
+		(end 151.794888 96)
 		(width 1.5)
 		(layer "B.Cu")
@@
 	)
 	(segment
-		(start 107 90)
-		(end 107 89.99)
+		(start 122.5 96)
+		(end 122.5 95.99)
 		(width 1.5)
 		(layer "B.Cu")
@@
 	)
 	(segment
-		(start 136.5 110.08)
-		(end 159.92 110.08)
+		(start 152 116.08)
+		(end 175.42 116.08)
 		(width 0.5)
 		(layer "F.Cu")
@@
 	)
 	(segment
-		(start 159.92 110.08)
-		(end 160 110)
+		(start 175.42 116.08)
+		(end 175.5 116)
 		(width 0.5)
 		(layer "F.Cu")
