File: Linear_Voltage_Regulator_5V.kicad_sch (KiCad schematic)
At the start: 8 parts, among them J1 INPUT 7-35V, J2 OUTPUT 5V, U1 L7805CV

Commit message: Task1: ajout rapport + BOM + nettoyage fichiers temporaires
Other:
- company: EUTech engineer -> EUTech engineers
Changed lines of the file:
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@@
 		(date "2026-03-02")
 		(rev "1.0")
-		(company "EUTech engineer")
+		(company "EUTech engineers")
 		(comment 1 "Regulator: L7805CV")
-		(comment 2 "Designer: Assane DIENG")
+		(comment 2 "Designer: Assane DIENG (Electrical Engineering Apprentice)")
 	)
 	(junction
